File: hardware/slow-cooker.sch (KiCad schematic (older format))
At the start: 54 parts, among them IC1 ATMEGA328-AN, P1 Input, P10 TEST_5V, P11 TEST_GND, P12 ICSP, P13 Output, P14 FTDI, P15 LCD 1, P16 LCD 2, P17 Temperature sensor, P2 TEST_19, P3 TEST_22, P4 TEST_23, P5 TEST_24, P6 TEST_25, P7 TEST_26, P8 TEST_27, P9 TEST_28, Q1 MMBT3904, SW1 Reset, SW2 TE D3223, U1 LT1761-3.3, U2 LS01-15B05S, X1 16MHz

Commit message: Board layout
Parts:
- removed L1: Wurth_744822301, Choke_Common-Mode_Wurth:CommonModeChoke_WuerthType-WE-CMB_Size-S, symbol Wurth_744822301
- removed P2: TEST_19, Connect:PINTST, symbol TST
- removed P3: TEST_22, Connect:PINTST, symbol TST
- removed P4: TEST_23, Connect:PINTST, symbol TST
- removed P5: TEST_24, Connect:PINTST, symbol TST
- removed P6: TEST_25, Connect:PINTST, symbol TST
- removed P7: TEST_26, Connect:PINTST, symbol TST
- removed P8: TEST_27, Connect:PINTST, symbol TST
- removed P9: TEST_28, Connect:PINTST, symbol TST
- added C18: 100n/400V/X, Capacitors_ThroughHole_Kemet:C_Rect_L24_W7.6_P20.3, symbol C_Small
- added F1: 10mA, Q, Fuse_Holders_and_Fuses:Fuseholder5x20_horiz_open_Schurter_0031_8201, symbol F_Small
- added L1: 1m/400V, Choke_Common-Mode_Epcos:CommonModeChoke_Epcos-B82730U, symbol EPCOSB82730U
- added L3: 1m/400V, Choke_Axial_ThroughHole:Choke_Horizontal_RM10mm, symbol L_Small
- added P18: Enclosure earth, Terminal_Blocks:TerminalBlock_Pheonix_MKDS1.5-2pol, symbol CONN_01X02
- P1: footprint Terminal_Blocks:TerminalBlock_Pheonix_MKDS1.5-3pol -> Connectors_Molex:Molex_MiniFit-JR-5556-04A_2x02x4.20mm_Straight; symbol CONN_01X03 -> CONN_02X02
- P13: footprint Terminal_Blocks:TerminalBlock_Pheonix_MKDS1.5-4pol -> Connectors_Molex:Molex_MiniFit-JR-5556-04A_2x02x4.20mm_Straight; symbol CONN_01X04 -> CONN_02X02
- P17: footprint Terminal_Blocks:TerminalBlock_Pheonix_MKDS1.5-3pol -> Terminal_Blocks:TerminalBlock_Pheonix_PT-3.5mm_3pol
- TVS1: renamed from 1.5KE300CA1; value TVS -> 1.5KE300CA1
Connections:
- net Earth_Protective: now also P1.1 (P1), P1.4 (P4), P13.4 (P4), P18.1 (P1), P18.2 (P2); no longer P1.3 (P3), P13.2 (P2)
- net Live: now also P1.2 (P2), F1.1; no longer P1.1 (P1), TVS1.1
- net Neutral: now also P1.3 (P3), L1.2 (IN-); no longer P1.2 (P2)
- net Relay_Neutral: now reaches P13.3 (P3), SW2.4
- net Relay_Live: now reaches SW2.7
- net Relay_Live: now also P13.2 (P2); no longer P13.4 (P4)
- net at C8.1, U2.1 (AC(N)): now also C18.2, L1.3 (OUT-)
- net at C7.2, U2.3 (AC(L)): now also L3.2
- new net: F1.2, L1.1 (IN+), TVS1.1
- new net: C18.1, L1.4 (OUT+), L3.1
- no-connect marks 4 -> 12
Other:
- note added: "Fuse holder cover:\nRS 337-1327"
- moved on the sheet: C10, C11, C12, C13, C16, C7, C8, D1, D2, L2, P10, P11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
